File: CapacityOfBattery.sch (KiCad schematic (older format))
At the start: 27 parts, among them J1 BATTERY, J2 DUT, Q1 IRLML6401TRPBF, Q2 IRLML6401TRPBF, Q3 IRLML6401TRPBF, Q4 IRLML6401TRPBF, Q5 SI2302, SW1 SW_Push, U1 NodeMCU1.0(ESP-12E)

Commit message: changed pcb layout
Parts:
- added R8: 30k, Resistor_SMD:R_0603_1608Metric_Pad1.05x0.95mm_HandSolder, symbol Device:R
- R7: value 60k -> 30k; footprint Resistor_SMD:R_0805_2012Metric_Pad1.15x1.40mm_HandSolder -> Resistor_SMD:R_0603_1608Metric_Pad1.05x0.95mm_HandSolder
- R9: renamed from R8; footprint Resistor_SMD:R_0805_2012Metric_Pad1.15x1.40mm_HandSolder -> Resistor_SMD:R_0603_1608Metric_Pad1.05x0.95mm_HandSolder
- gave numbers to parts that had none: 2
- renumbered R9 to R10, RL2 to RL3, RL3 to RL5
Connections:
- net Vin: now also R8.2; no longer R7.2
- new net: R7.2, R8.1
Other:
- moved on the sheet: Q5, R6, R9
Changed lines of the file:
@@
 $EndComp
 $Comp
-L Device:R RL2
+L Device:R RL3
 U 1 1 5D049EE8
 P 4250 2800
-F 0 "RL2" V 4350 2750 50  0000 L CNN
+F 0 "RL3" V 4350 2750 50  0000 L CNN
 F 1 "232" V 4250 2700 50  0000 L CNN
 F 2 "Resistor_SMD:R_0805_2012Metric_Pad1.15x1.40mm_HandSolder" V 4180 2800 50  0001 C CNN
@@
 $EndComp
 $Comp
-L Device:R RL3
+L Device:R RL5
 U 1 1 5D049F1F
 P 5600 2800
-F 0 "RL3" V 5700 2750 50  0000 L CNN
+F 0 "RL5" V 5700 2750 50  0000 L CNN
 F 1 "232" V 5600 2700 50  0000 L CNN
 F 2 "Resistor_SMD:R_0805_2012Metric_Pad1.15x1.40mm_HandSolder" V 5530 2800 50  0001 C CNN
@@
 	6500 2300 6500 2050
 $Comp
-L power:GND #PWR05
+L power:GND #PWR07
 U 1 1 5D04B406
 P 9100 1400
-F 0 "#PWR05" H 9100 1150 50  0001 C CNN
+F 0 "#PWR07" H 9100 1150 50  0001 C CNN
 F 1 "GND" H 9105 1227 50  0000 C CNN
 F 2 "" H 9100 1400 50  0001 C CNN
@@
 En_VD
 $Comp
-L Device:R R7
-U 1 1 5D0CB5DD
-P 8750 4300
-F 0 "R7" H 8820 4346 50  0000 L CNN
-F 1 "60k" H 8820 4255 50  0000 L CNN
-F 2 "Resistor_SMD:R_0805_2012Metric_Pad1.15x1.40mm_HandSolder" V 8680 4300 50  0001 C CNN
-F 3 "~" H 8750 4300 50  0001 C CNN
-	1    8750 4300
-	1    0    0    -1
-$EndComp
-$Comp
-L Device:R R8
+L Device:R R9
 U 1 1 5D0CB64B
-P 8750 4750
-F 0 "R8" H 8820 4796 50  0000 L CNN
-F 1 "30k" H 8820 4705 50  0000 L CNN
-F 2 "Resistor_SMD:R_0805_2012Metric_Pad1.15x1.40mm_HandSolder" V 8680 4750 50  0001 C CNN
-F 3 "~" H 8750 4750 50  0001 C CNN
-	1    8750 4750
+P 8750 5100
+F 0 "R9" V 8850 5050 50  0000 L CNN
+F 1 "30k" V 8750 5000 50  0000 L CNN
+F 2 "Resistor_SMD:R_0603_1608Metric_Pad1.05x0.95mm_HandSolder" V 8680 5100 50  0001 C CNN
+F 3 "~" H 8750 5100 50  0001 C CNN
+	1    8750 5100
 	1    0    0    -1
 $EndComp
@@
 L Transistor_FET_SI2302:SI2302 Q5
 U 1 1 5D0CB6CC
-P 8750 5250
-F 0 "Q5" H 8849 5296 50  0000 L CNN
-F 1 "SI2302" H 8849 5205 50  0000 L CNN
-F 2 "Package_TO_SOT_SMD:SOT-23" H 8550 5550 50  0001 C CNN
-F 3 "" H 8550 5550 50  0001 C CNN
-	1    8750 5250
-	1    0    0    -1
-$EndComp
-$Comp
-L power:GND #PWR06
+P 8750 5600
+F 0 "Q5" H 8849 5646 50  0000 L CNN
+F 1 "SI2302" H 8849 5555 50  0000 L CNN
+F 2 "Package_TO_SOT_SMD:SOT-23" H 8550 5900 50  0001 C CNN
+F 3 "" H 8550 5900 50  0001 C CNN
+	1    8750 5600
+	1    0    0    -1
+$EndComp
+$Comp
+L power:GND #PWR05
 U 1 1 5D0CB735
-P 8750 5550
-F 0 "#PWR06" H 8750 5300 50  0001 C CNN
-F 1 "GND" H 8755 5377 50  0000 C CNN
-F 2 "" H 8750 5550 50  0001 C CNN
-F 3 "" H 8750 5550 50  0001 C CNN
-	1    8750 5550
-	1    0    0    -1
-$EndComp
-Wire Wire Line
-	8750 4450 8750 4550
-Wire Wire Line
-	8750 4900 8750 5050
-Wire Wire Line
-	8750 5450 8750 5500
+P 8750 5900
+F 0 "#PWR05" H 8750 5650 50  0001 C CNN
+F 1 "GND" H 8755 5727 50  0000 C CNN
+F 2 "" H 8750 5900 50  0001 C CNN
+F 3 "" H 8750 5900 50  0001 C CNN
+	1    8750 5900
+	1    0    0    -1
+$EndComp
+Wire Wire Line
+	8750 4800 8750 4900
+Wire Wire Line
+	8750 5250 8750 5400
+Wire Wire Line
+	8750 5800 8750 5850
 Wire Wire Line
 	8500 4050 8750 4050
@@
 Text Label 8500 4050 0    50   ~ 0
 Vbat
-Text Label 7900 5250 0    50   ~ 0
+Text Label 7900 5600 0    50   ~ 0
 En_VD
 Wire Wire Line
-	8750 4550 8500 4550
-Connection ~ 8750 4550
-Wire Wire Line
-	8750 4550 8750 4600
-Text Label 8500 4550 0    50   ~ 0
+	8750 4900 8500 4900
+Connection ~ 8750 4900
+Wire Wire Line
+	8750 4900 8750 4950
+Text Label 8500 4900 0    50   ~ 0
 Vin
 Text Notes 4900 3950 0    50   ~ 0
@@
 L Device:R R6
 U 1 1 5D0F6D0C
-P 8300 5500
-F 0 "R6" V 8400 5500 50  0000 C CNN
-F 1 "10k" V 8300 5500 50  0000 C CNN
-F 2 "Resistor_SMD:R_0805_2012Metric_Pad1.15x1.40mm_HandSolder" V 8230 5500 50  0001 C CNN
-F 3 "~" H 8300 5500 50  0001 C CNN
-	1    8300 5500
+P 8300 5850
+F 0 "R6" V 8400 5850 50  0000 C CNN
+F 1 "10k" V 8300 5850 50  0000 C CNN
+F 2 "Resistor_SMD:R_0805_2012Metric_Pad1.15x1.40mm_HandSolder" V 8230 5850 50  0001 C CNN
+F 3 "~" H 8300 5850 50  0001 C CNN
+	1    8300 5850
 	0    1    1    0
 $EndComp
 Wire Wire Line
-	8450 5500 8750 5500
-Connection ~ 8750 5500
-Wire Wire Line
-	8750 5500 8750 5550
-Wire Wire Line
-	8150 5500 8150 5250
-Wire Wire Line
-	8150 5250 8450 5250
+	8450 5850 8750 5850
+Connection ~ 8750 5850
+Wire Wire Line
+	8750 5850 8750 5900
+Wire Wire Line
+	8150 5850 8150 5600
+Wire Wire Line
+	8150 5600 8450 5600
 Wire Wire Line
 	2900 2500 2900 2600
@@
 Wire Wire Line
 	6500 5200 6750 5200
-Connection ~ 8150 5250
-Wire Wire Line
-	7900 5250 8150 5250
+Connection ~ 8150 5600
+Wire Wire Line
+	7900 5600 8150 5600
 Text Label 2800 4300 0    50   ~ 0
 LED1
@@
 $EndComp
 $Comp
-L Device:R R9
+L Device:R R10
 U 1 1 5D1A9944
 P 8800 2950
-F 0 "R9" H 8870 2996 50  0000 L CNN
-F 1 "1k" H 8870 2905 50  0000 L CNN
+F 0 "R10" V 8900 2900 50  0000 L CNN
+F 1 "1k" V 8800 2900 50  0000 L CNN
 F 2 "Resistor_SMD:R_0805_2012Metric_Pad1.15x1.40mm_HandSolder" V 8730 2950 50  0001 C CNN
 F 3 "~" H 8800 2950 50  0001 C CNN
@@
 	8800 2650 8800 2700
 $Comp
-L power:GND #PWR0101
+L power:GND #PWR06
 U 1 1 5D1B375E
 P 8800 3200
-F 0 "#PWR0101" H 8800 2950 50  0001 C CNN
+F 0 "#PWR06" H 8800 2950 50  0001 C CNN
 F 1 "GND" H 8805 3027 50  0000 C CNN
 F 2 "" H 8800 3200 50  0001 C CNN
@@
 A switch is used \nto select the load\n(Active HIGH)
 $Comp
-L Device:R RL?
+L Device:R RL2
 U 1 1 5D0C89B4
 P 2900 3100
-F 0 "RL?" V 3000 3050 50  0000 L CNN
+F 0 "RL2" V 3000 3050 50  0000 L CNN
 F 1 "232" V 2900 3000 50  0000 L CNN
 F 2 "Resistor_SMD:R_0805_2012Metric_Pad1.15x1.40mm_HandSolder" V 2830 3100 50  0001 C CNN
@@
 	2900 2950 2900 2900
 $Comp
-L Device:R RL?
+L Device:R RL4
 U 1 1 5D0CC57E
 P 5350 2800
-F 0 "RL?" V 5450 2750 50  0000 L CNN
+F 0 "RL4" V 5450 2750 50  0000 L CNN
 F 1 "232" V 5350 2700 50  0000 L CNN
 F 2 "Resistor_SMD:R_0805_2012Metric_Pad1.15x1.40mm_HandSolder" V 5280 2800 50  0001 C CNN
@@
 Wire Wire Line
 	5600 3000 5600 3050
+$Comp
+L Device:R R7
+U 1 1 5D0DAE27
+P 8750 4300
+F 0 "R7" V 8850 4250 50  0000 L CNN
+F 1 "30k" V 8750 4200 50  0000 L CNN
+F 2 "Resistor_SMD:R_0603_1608Metric_Pad1.05x0.95mm_HandSolder" V 8680 4300 50  0001 C CNN
+F 3 "~" H 8750 4300 50  0001 C CNN
+	1    8750 4300
+	1    0    0    -1
+$EndComp
+$Comp
+L Device:R R8
+U 1 1 5D0DCF90
+P 8750 4650
+F 0 "R8" V 8850 4600 50  0000 L CNN
+F 1 "30k" V 8750 4550 50  0000 L CNN
+F 2 "Resistor_SMD:R_0603_1608Metric_Pad1.05x0.95mm_HandSolder" V 8680 4650 50  0001 C CNN
+F 3 "~" H 8750 4650 50  0001 C CNN
+	1    8750 4650
+	1    0    0    -1
+$EndComp
+Wire Wire Line
+	8750 4500 8750 4450
 $EndSCHEMATC
