File: CapacityOfBattery.sch (KiCad schematic (older format))
At the start: 28 parts, among them J1 BATTERY, J2 DUT, Q1 IRLML6401TRPBF, Q2 IRLML6401TRPBF, Q3 IRLML6401TRPBF, Q4 IRLML6401TRPBF, Q5 SI2302, SW1 SW_Push, U1 NodeMCU1.0(ESP-12E)

Commit message: pcb updated
Parts:
- added H1, H2, H3, H4: MountingHole, MountingHole:MountingHole_3.2mm_M3_ISO7380, symbol Mechanical:MountingHole
Changed lines of the file:
@@
 Wire Wire Line
 	8750 4500 8750 4450
+$Comp
+L Mechanical:MountingHole H1
+U 1 1 5D0C9E38
+P 1500 3600
+F 0 "H1" H 1600 3646 50  0000 L CNN
+F 1 "MountingHole" H 1600 3555 50  0000 L CNN
+F 2 "MountingHole:MountingHole_3.2mm_M3_ISO7380" H 1500 3600 50  0001 C CNN
+F 3 "~" H 1500 3600 50  0001 C CNN
+	1    1500 3600
+	1    0    0    -1
+$EndComp
+$Comp
+L Mechanical:MountingHole H2
+U 1 1 5D0C9EE2
+P 1500 3850
+F 0 "H2" H 1600 3896 50  0000 L CNN
+F 1 "MountingHole" H 1600 3805 50  0000 L CNN
+F 2 "MountingHole:MountingHole_3.2mm_M3_ISO7380" H 1500 3850 50  0001 C CNN
+F 3 "~" H 1500 3850 50  0001 C CNN
+	1    1500 3850
+	1    0    0    -1
+$EndComp
+$Comp
+L Mechanical:MountingHole H3
+U 1 1 5D0CC0E0
+P 1500 4100
+F 0 "H3" H 1600 4146 50  0000 L CNN
+F 1 "MountingHole" H 1600 4055 50  0000 L CNN
+F 2 "MountingHole:MountingHole_3.2mm_M3_ISO7380" H 1500 4100 50  0001 C CNN
+F 3 "~" H 1500 4100 50  0001 C CNN
+	1    1500 4100
+	1    0    0    -1
+$EndComp
+$Comp
+L Mechanical:MountingHole H4
+U 1 1 5D0CE2E5
+P 1500 4350
+F 0 "H4" H 1600 4396 50  0000 L CNN
+F 1 "MountingHole" H 1600 4305 50  0000 L CNN
+F 2 "MountingHole:MountingHole_3.2mm_M3_ISO7380" H 1500 4350 50  0001 C CNN
+F 3 "~" H 1500 4350 50  0001 C CNN
+	1    1500 4350
+	1    0    0    -1
+$EndComp
 $EndSCHEMATC
