File: CapacityOfBattery.kicad_pcb (KiCad board)
At the start: 2 copper layers, 30.5 x 57.1 mm, 21 parts, among them J1 BATTERY, J2 DUT, Q1 IRLML6401TRPBF, Q2 IRLML6401TRPBF, Q3 IRLML6401TRPBF, Q4 IRLML6401TRPBF, Q5 IRLML6401TRPBF

Commit message: updated pcb
Parts:
- removed ?: For LOLin (NodeMCU v3), SUDHEENDRA_HEGDE:NodeMCU-LoLinV3
- removed ? (x4): MountingHole, MountingHole:MountingHole_3.2mm_M3
- added D1: LED, LED_SMD:LED_0805_2012Metric_Pad1.15x1.40mm_HandSolder, F.Cu at (19.5, 65.2)
- added D2: LED, LED_SMD:LED_0805_2012Metric_Pad1.15x1.40mm_HandSolder, F.Cu at (24.1, 65.2)
- added D3: LED, LED_SMD:LED_0805_2012Metric_Pad1.15x1.40mm_HandSolder, F.Cu at (28.7, 65.2)
- added D4: LED, LED_SMD:LED_0805_2012Metric_Pad1.15x1.40mm_HandSolder, F.Cu at (33.3, 65.2)
- added D5: LED, LED_SMD:LED_0805_2012Metric_Pad1.15x1.40mm_HandSolder, F.Cu at (37.9, 65.2)
- added Q6: SI2302, Package_TO_SOT_SMD:SOT-23, F.Cu at (28.7, 25.4)
- added R6: 560, Resistor_SMD:R_0805_2012Metric_Pad1.15x1.40mm_HandSolder, F.Cu at (33.7, 61.0)
- added R7: 60k, Resistor_SMD:R_0805_2012Metric_Pad1.15x1.40mm_HandSolder, F.Cu at (23.6, 27.9)
- added R8: 30k, Resistor_SMD:R_0805_2012Metric_Pad1.15x1.40mm_HandSolder, F.Cu at (23.6, 24.1)
- added R9: 10k, Resistor_SMD:R_0805_2012Metric_Pad1.15x1.40mm_HandSolder, F.Cu at (33.7, 26.6)
- added U1: NodeMCU1.0(ESP-12E), SUDHEENDRA_HEGDE:NodeMCU-LoLinV3, F.Cu at (28.5, 43.6)
- moved J1 76.4 mm to (35.6, 19.1), turned to 270 degrees
- moved J2 76.4 mm to (24.1, 19.1), turned to 270 degrees
- moved R5 29.3 mm to (33.7, 57.1), turned to 180 degrees
- moved Q5 29.2 mm to (28.7, 58.4)
- moved Q4 26.9 mm to (28.7, 52.0)
- moved Q3 25.7 mm to (28.7, 45.7)
- moved RL4 25.2 mm to (23.6, 52.0)
- moved Q2 24.6 mm to (28.7, 39.4)
- moved R4 24.3 mm to (33.7, 53.3), turned to 180 degrees
- moved RL3 24.0 mm to (23.6, 45.7)
- moved Q1 23.5 mm to (28.7, 33.0)
- moved R3 23.0 mm to (33.7, 47.0), turned to 180 degrees
- moved RL2 22.9 mm to (23.6, 39.4)
- moved RL1 21.8 mm to (23.6, 33.0)
- moved R2 21.7 mm to (33.7, 40.6), turned to 180 degrees
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Routing:
- net /Ctrl1: track 14.9 -> 60.7 mm, vias 0 -> 2
- net /Ctrl2: track 16.7 -> 56.9 mm, vias 0 -> 2
- net /Ctrl3: track 20.3 -> 53.3 mm, vias 0 -> 2
- net GND: track 0.00 -> 28.8 mm
- net /Vcc: track 62.5 -> 35.3 mm, vias 4 -> 0
- net Net-(J2-Pad2): track 19.1 -> 44.7 mm, vias 0 -> 1
- net /En_VoltageDivider: track 0.00 -> 24.2 mm
- net Net-(D1-Pad2): track 0.00 -> 21.9 mm
- net /Ctrl5: track 17.2 -> 35.5 mm, vias 0 -> 2
- net /Vbat: track 86.1 -> 72.6 mm
- net /Ctrl4: track 26.9 -> 40.0 mm, vias 1 -> 2
- net /Vin: track 0.00 -> 12.2 mm
- net Net-(Q6-Pad3): track 0.00 -> 3.58 mm
- net Net-(Q2-Pad3): track 4.85 -> 3.05 mm
- net Net-(Q4-Pad3): track 4.85 -> 3.05 mm
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Other:
- board size 30.5 x 57.1 mm -> 31.8 x 58.4 mm
- board text added: "DUT"
- board text added: "LD1 560"
- board text added: "LD2 232"
- board text added: "LD3 116"
- board text added: "LD4 047"

Commit message: updated pcb
Parts:
- RL2: value 330 -> 232
- RL3: value 100 -> 116
Connections:
- U1 pad 10: GND -> Net-(U1-Pad10)
- U1 pad 11: (no net) -> /Vcc
- U1 pad 17: GND -> Net-(U1-Pad17)
- U1 pad 2: GND -> Net-(U1-Pad2)
- U1 pad 24: GND -> Net-(U1-Pad24)
- U1 pad 25: (no net) -> Net-(U1-Pad25)
Changed lines of the file:
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@@
     (zones 0)
     (modules 27)
-    (nets 33)
+    (nets 38)
   )
   (page A4)
@@
   (net 31 "Net-(D1-Pad2)")
   (net 32 "Net-(J2-Pad2)")
+  (net 33 "Net-(U1-Pad25)")
+  (net 34 "Net-(U1-Pad24)")
+  (net 35 "Net-(U1-Pad17)")
+  (net 36 "Net-(U1-Pad10)")
+  (net 37 "Net-(U1-Pad2)")
   (net_class Default "This is the default net class."
     (clearance 0.5)
@@
     (add_net "Net-(Q4-Pad3)")
     (add_net "Net-(Q6-Pad3)")
+    (add_net "Net-(U1-Pad10)")
     (add_net "Net-(U1-Pad12)")
     (add_net "Net-(U1-Pad13)")
     (add_net "Net-(U1-Pad15)")
+    (add_net "Net-(U1-Pad17)")
     (add_net "Net-(U1-Pad18)")
     (add_net "Net-(U1-Pad19)")
+    (add_net "Net-(U1-Pad2)")
     (add_net "Net-(U1-Pad23)")
+    (add_net "Net-(U1-Pad24)")
+    (add_net "Net-(U1-Pad25)")
     (add_net "Net-(U1-Pad26)")
     (add_net "Net-(U1-Pad27)")
@@
     (pad 26 thru_hole circle (at 13.97 -10.16) (size 1.524 1.524) (drill 0.762) (layers *.Cu *.Mask F.SilkS)
       (net 5 "Net-(U1-Pad26)"))
-    (pad 25 thru_hole circle (at 13.97 -7.62) (size 1.524 1.524) (drill 0.762) (layers *.Cu *.Mask F.SilkS))
+    (pad 25 thru_hole circle (at 13.97 -7.62) (size 1.524 1.524) (drill 0.762) (layers *.Cu *.Mask F.SilkS)
+      (net 33 "Net-(U1-Pad25)"))
     (pad 24 thru_hole circle (at 13.97 -5.08) (size 1.524 1.524) (drill 0.762) (layers *.Cu *.Mask F.SilkS)
-      (net 11 GND))
+      (net 34 "Net-(U1-Pad24)"))
     (pad 23 thru_hole circle (at 13.97 -2.54) (size 1.524 1.524) (drill 0.762) (layers *.Cu *.Mask F.SilkS)
       (net 6 "Net-(U1-Pad23)"))
@@
       (net 9 "Net-(U1-Pad18)"))
     (pad 17 thru_hole circle (at 13.97 12.7) (size 1.524 1.524) (drill 0.762) (layers *.Cu *.Mask F.SilkS)
-      (net 11 GND))
+      (net 35 "Net-(U1-Pad17)"))
     (pad 16 thru_hole circle (at 13.97 15.24) (size 1.524 1.524) (drill 0.762) (layers *.Cu *.Mask F.SilkS)
       (net 14 /Vcc))
@@
     (pad 12 thru_hole circle (at -13.97 7.62) (size 1.524 1.524) (drill 0.762) (layers *.Cu *.Mask F.SilkS)
       (net 13 "Net-(U1-Pad12)"))
-    (pad 11 thru_hole circle (at -13.97 5.08) (size 1.524 1.524) (drill 0.762) (layers *.Cu *.Mask F.SilkS))
+    (pad 11 thru_hole circle (at -13.97 5.08) (size 1.524 1.524) (drill 0.762) (layers *.Cu *.Mask F.SilkS)
+      (net 14 /Vcc))
     (pad 10 thru_hole circle (at -13.97 2.54) (size 1.524 1.524) (drill 0.762) (layers *.Cu *.Mask F.SilkS)
-      (net 11 GND))
+      (net 36 "Net-(U1-Pad10)"))
     (pad 9 thru_hole circle (at -13.97 0) (size 1.524 1.524) (drill 0.762) (layers *.Cu *.Mask F.SilkS)
       (net 15 "Net-(U1-Pad9)"))
@@
       (net 21 "Net-(U1-Pad3)"))
     (pad 2 thru_hole circle (at -13.97 -17.78) (size 1.524 1.524) (drill 0.762) (layers *.Cu *.Mask F.SilkS)
-      (net 11 GND))
+      (net 37 "Net-(U1-Pad2)"))
     (pad 1 thru_hole circle (at -13.97 -20.32) (size 1.524 1.524) (drill 0.762) (layers *.Cu *.Mask F.SilkS)
       (net 29 /Vin))
@@
       (effects (font (size 1 1) (thickness 0.15)))
     )
-    (fp_text value 330 (at 0 1.65) (layer F.Fab)
+    (fp_text value 232 (at 0 1.65) (layer F.Fab)
       (effects (font (size 1 1) (thickness 0.15)))
     )
@@
       (effects (font (size 1 1) (thickness 0.15)))
     )
-    (fp_text value 100 (at 0 1.65) (layer F.Fab)
+    (fp_text value 116 (at 0 1.65) (layer F.Fab)
       (effects (font (size 1 1) (thickness 0.15)))
     )
@@
     (effects (font (size 1 1) (thickness 0.15)))
   )
-  (via (at 31.75 59.055) (size 0.8) (drill 0.4) (layers F.Cu B.Cu) (net 7))
   (via (at 21.59 67.31) (size 0.8) (drill 0.4) (layers F.Cu B.Cu) (net 1))
-  (via (at 26.67 67.31) (size 0.8) (drill 0.4) (layers F.Cu B.Cu) (net 2))
-  (via (at 30.48 67.31) (size 0.8) (drill 0.4) (layers F.Cu B.Cu) (net 3))
-  (via (at 40.64 64.77) (size 0.8) (drill 0.4) (layers F.Cu B.Cu) (net 7))
-  (via (at 35.56 67.31) (size 0.8) (drill 0.4) (layers F.Cu B.Cu) (net 4))
-  (via (at 25.4 58.42) (size 0.8) (drill 0.4) (layers F.Cu B.Cu) (net 32))
-  (via (at 33.02 38.1) (size 0.8) (drill 0.4) (layers F.Cu B.Cu) (net 2))
-  (via (at 33.02 44.45) (size 0.8) (drill 0.4) (layers F.Cu B.Cu) (net 3))
-  (via (at 33.02 50.8) (size 0.8) (drill 0.4) (layers F.Cu B.Cu) (net 4))
   (segment (start 32.395 33.95) (end 32.715 34.27) (width 0.5) (layer F.Cu) (net 1))
   (segment (start 29.66 33.95) (end 32.395 33.95) (width 0.5) (layer F.Cu) (net 1))
@@
   (segment (start 32.715 33.035) (end 32.73 33.02) (width 0.5) (layer F.Cu) (net 1))
   (segment (start 32.715 34.27) (end 32.715 33.035) (width 0.5) (layer F.Cu) (net 1))
+  (via (at 26.67 67.31) (size 0.8) (drill 0.4) (layers F.Cu B.Cu) (net 2))
+  (via (at 33.02 38.1) (size 0.8) (drill 0.4) (layers F.Cu B.Cu) (net 2))
   (segment (start 32.395 40.3) (end 32.715 40.62) (width 0.5) (layer F.Cu) (net 2))
   (segment (start 29.66 40.3) (end 32.395 40.3) (width 0.5) (layer F.Cu) (net 2))
@@
   (segment (start 25.175899 67.31) (end 24.100833 66.234934) (width 0.5) (layer F.Cu) (net 2))
   (segment (start 26.67 67.31) (end 25.175899 67.31) (width 0.5) (layer F.Cu) (net 2))
+  (via (at 30.48 67.31) (size 0.8) (drill 0.4) (layers F.Cu B.Cu) (net 3))
+  (via (at 33.02 44.45) (size 0.8) (drill 0.4) (layers F.Cu B.Cu) (net 3))
   (segment (start 32.395 46.65) (end 32.715 46.97) (width 0.5) (layer F.Cu) (net 3))
   (segment (start 29.66 46.65) (end 32.395 46.65) (width 0.5) (layer F.Cu) (net 3))
@@
   (segment (start 29.775899 67.31) (end 28.700833 66.234934) (width 0.5) (layer F.Cu) (net 3))
   (segment (start 30.48 67.31) (end 29.775899 67.31) (width 0.5) (layer F.Cu) (net 3))
+  (via (at 35.56 67.31) (size 0.8) (drill 0.4) (layers F.Cu B.Cu) (net 4))
+  (via (at 33.02 50.8) (size 0.8) (drill 0.4) (layers F.Cu B.Cu) (net 4))
   (segment (start 32.395 53) (end 32.715 53.32) (width 0.5) (layer F.Cu) (net 4))
   (segment (start 29.66 53) (end 32.395 53) (width 0.5) (layer F.Cu) (net 4))
@@
   (segment (start 34.375899 67.31) (end 33.300833 66.234934) (width 0.5) (layer F.Cu) (net 4))
   (segment (start 35.56 67.31) (end 34.375899 67.31) (width 0.5) (layer F.Cu) (net 4))
+  (via (at 31.75 59.055) (size 0.8) (drill 0.4) (layers F.Cu B.Cu) (net 7))
+  (via (at 40.64 64.77) (size 0.8) (drill 0.4) (layers F.Cu B.Cu) (net 7))
   (segment (start 42.47 48.97) (end 42.47 48.68) (width 0.5) (layer B.Cu) (net 7))
   (segment (start 39.175066 66.234934) (end 37.900833 66.234934) (width 0.5) (layer F.Cu) (net 7))
@@
   (segment (start 22.555 33) (end 22.555 39.35) (width 0.5) (layer F.Cu) (net 11))
   (segment (start 22.555 39.35) (end 22.555 45.7) (width 0.5) (layer F.Cu) (net 11))
-  (via (at 25.4 30.48) (size 0.8) (drill 0.4) (layers F.Cu B.Cu) (net 22))
-  (via (at 25.4 36.83) (size 0.8) (drill 0.4) (layers F.Cu B.Cu) (net 22))
-  (via (at 25.4 43.18) (size 0.8) (drill 0.4) (layers F.Cu B.Cu) (net 22))
-  (via (at 25.4 49.53) (size 0.8) (drill 0.4) (layers F.Cu B.Cu) (net 22))
-  (via (at 25.4 55.88) (size 0.8) (drill 0.4) (layers F.Cu B.Cu) (net 22))
   (segment (start 34.765 57.15) (end 34.765 60.96) (width 0.5) (layer F.Cu) (net 14))
   (segment (start 40.35 60.96) (end 42.47 58.84) (width 0.5) (layer F.Cu) (net 14))
@@
   (segment (start 34.765 34.27) (end 34.765 40.62) (width 0.5) (layer F.Cu) (net 14))
   (segment (start 34.765 57.15) (end 34.765 53.32) (width 0.5) (layer F.Cu) (net 14))
+  (via (at 25.4 30.48) (size 0.8) (drill 0.4) (layers F.Cu B.Cu) (net 22))
+  (via (at 25.4 36.83) (size 0.8) (drill 0.4) (layers F.Cu B.Cu) (net 22))
+  (via (at 25.4 43.18) (size 0.8) (drill 0.4) (layers F.Cu B.Cu) (net 22))
+  (via (at 25.4 49.53) (size 0.8) (drill 0.4) (layers F.Cu B.Cu) (net 22))
+  (via (at 25.4 55.88) (size 0.8) (drill 0.4) (layers F.Cu B.Cu) (net 22))
   (segment (start 29.66 31.15) (end 29.66 32.05) (width 0.5) (layer F.Cu) (net 22))
   (segment (start 24.605 27.94) (end 26.45 27.94) (width 0.5) (layer F.Cu) (net 22))
@@
   (segment (start 19.500833 64.184934) (end 24.100833 64.184934) (width 0.5) (layer F.Cu) (net 31))
   (segment (start 24.100833 64.184934) (end 28.700833 64.184934) (width 0.5) (layer F.Cu) (net 31))
+  (via (at 25.4 58.42) (size 0.8) (drill 0.4) (layers F.Cu B.Cu) (net 32))
   (segment (start 27.64 58.42) (end 27.66 58.4) (width 0.5) (layer F.Cu) (net 32))
   (segment (start 25.4 58.42) (end 27.64 58.42) (width 0.5) (layer F.Cu) (net 32))

Commit message: modified PCB
Parts:
- added ?: MountingHole, MountingHole:MountingHole_3.2mm_M3, F.Cu at (41.2, 67.7)
- added ?: MountingHole, MountingHole:MountingHole_3.2mm_M3, F.Cu at (15.8, 67.7)
- added ?: MountingHole, MountingHole:MountingHole_3.2mm_M3, F.Cu at (15.8, 15.7)
- added ?: MountingHole, MountingHole:MountingHole_3.2mm_M3, F.Cu at (41.2, 15.7)
- moved J1 2.54 mm to (33.0, 19.1), turned to 90 degrees
- moved J2 2.54 mm to (21.6, 19.1), turned to 90 degrees
- moved D5 2.31 mm to (35.7, 65.9)
- moved D1 1.93 mm to (21.3, 65.9)
- moved D4 1.38 mm to (32.1, 65.9)
- moved D2 1.06 mm to (24.9, 65.9)
- moved D3 0.72 mm to (28.5, 65.9)
Connections:
- U1 pad 10: Net-(U1-Pad10) -> GND
- U1 pad 17: Net-(U1-Pad17) -> GND
- U1 pad 2: Net-(U1-Pad2) -> GND
- U1 pad 24: Net-(U1-Pad24) -> GND
Routing:
- net Net-(D1-Pad2): track 21.9 -> 18.6 mm
- net /Ctrl5: track 35.5 -> 33.1 mm
- net /Ctrl1: track 60.7 -> 62.7 mm
- net /Ctrl2: track 56.9 -> 58.0 mm
- net Net-(J2-Pad2): track 44.7 -> 45.8 mm
- net /Vbat: track 72.6 -> 73.7 mm
- net /Ctrl4: track 40.0 -> 39.3 mm
- net /Ctrl3: track 53.3 -> 53.9 mm
Other:
- board text added: "047"
- board text added: "116"
- board text added: "232"
- board text added: "560"
- board text removed: "LD1 560"
- board text removed: "LD2 232"
- board text removed: "LD3 116"
- board text removed: "LD4 047"

Commit message: update pcb
Parts:
- removed the ? at (41.2, 67.7)
- removed the ? at (15.8, 67.7)
- removed the ? at (15.8, 15.7)
- removed the ? at (41.2, 15.7)
- removed D5: LED, LED_SMD:LED_0805_2012Metric_Pad1.15x1.40mm_HandSolder
- removed Q6: SI2302, Package_TO_SOT_SMD:SOT-23
- removed RL4: 47, Resistor_SMD:R_0805_2012Metric_Pad1.15x1.40mm_HandSolder
- removed U1: NodeMCU1.0(ESP-12E), SUDHEENDRA_HEGDE:NodeMCU-LoLinV3
- added ?: NodeMCU1.0(ESP-12E), SUDHEENDRA_HEGDE:NodeMCU-LoLinV3, F.Cu at (29.2, 43.2)
- added SW1: SW_Push, Button_Switch_THT:SW_PUSH_6mm, F.Cu at (104.1, 36.8)
- D1, D2, D3, D4: moved to B.Cu
- Q5: value IRLML6401TRPBF -> SI2302
- R2: value 100k -> 560
- R6: value 560 -> 10k
- R9: value 10k -> 1k
- moved R9 73.6 mm to (64.1, 93.7), turned to 0 degrees
- moved D1 46.7 mm to (39.4, 22.9), turned to 180 degrees
- moved D2 43.0 mm to (39.4, 25.4), turned to 180 degrees
- moved D3 39.5 mm to (39.4, 27.9), turned to 180 degrees
- moved D4 36.2 mm to (39.4, 30.5), turned to 180 degrees
- moved R6 28.0 mm to (35.0, 33.0)
- moved Q5 26.7 mm to (29.9, 31.8)
- moved R5 20.2 mm to (35.0, 36.9)
- moved Q1 19.1 mm to (29.6, 52.1)
- moved RL1 15.3 mm to (24.9, 48.2), turned to 180 degrees
- moved Q4 15.3 mm to (29.9, 36.8)
- moved R4 14.5 mm to (35.0, 38.9)
- moved R1 8.64 mm to (35.0, 42.8)
- moved Q2 7.70 mm to (29.6, 47.0)
- moved R8 6.40 mm to (24.9, 30.4)
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Connections:
- D1 pad 1: /Ctrl1 -> /LED1
- D2 pad 1: /Ctrl2 -> /LED2
- D3 pad 1: /Ctrl3 -> /LED3
- D4 pad 1: /Ctrl4 -> /LED4
- J2 pad 2: Net-(J2-Pad2) -> /dut
- Q4 pad 3: Net-(Q4-Pad3) -> /dut
- Q5 pad 1: /Ctrl5 -> /En_VD
- Q5 pad 2: /Vbat -> GND
- Q5 pad 3: Net-(J2-Pad2) -> Net-(Q5-Pad3)
- R2 pad 2: /Ctrl2 -> Net-(D1-Pad2)
- R3 pad 2: /Ctrl3 -> /Ctrl2
- R4 pad 2: /Ctrl4 -> /Ctrl3
- R5 pad 2: /Ctrl5 -> /Ctrl4
- R6 pad 1: /Vcc -> GND
- R6 pad 2: Net-(D1-Pad2) -> /En_VD
- R8 pad 2: Net-(Q6-Pad3) -> Net-(Q5-Pad3)
- R9 pad 1: GND -> /SW
- R9 pad 2: /En_VoltageDivider -> GND
- RL1 pad 1: GND -> Net-(Q1-Pad3)
- RL1 pad 2: Net-(Q1-Pad3) -> GND
- RL2 pad 1: GND -> Net-(Q2-Pad3)
- RL2 pad 2: Net-(Q2-Pad3) -> GND
- RL3 pad 1: GND -> Net-(Q3-Pad3)
- RL3 pad 2: Net-(Q3-Pad3) -> GND
Routing:
- net /Vbat: track 73.7 -> 0.00 mm, vias 5 -> 0
- net /Ctrl1: track 62.7 -> 0.00 mm, vias 2 -> 0
- net /Ctrl2: track 58.0 -> 0.00 mm, vias 2 -> 0
- net /Ctrl3: track 53.9 -> 0.00 mm, vias 2 -> 0
- net Net-(J2-Pad2): track 45.8 -> 0.00 mm, vias 1 -> 0
- net /Ctrl4: track 39.3 -> 0.00 mm, vias 2 -> 0
- net /Vcc: track 35.3 -> 0.00 mm
- net /Ctrl5: track 33.1 -> 0.00 mm, vias 2 -> 0
- net GND: track 28.8 -> 0.00 mm
- net /En_VoltageDivider: track 24.2 -> 0.00 mm
- net Net-(D1-Pad2): track 18.6 -> 0.00 mm
- net /Vin: track 12.2 -> 0.00 mm
- net Net-(Q6-Pad3): track 3.58 -> 0.00 mm
- net Net-(Q3-Pad3): track 3.32 -> 0.00 mm
- net Net-(Q4-Pad3): track 3.05 -> 0.00 mm
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- removed copper zone on B.Cu, net GND
- removed copper zone on F.Cu, net GND
Other:
- board outline removed
- board text removed: "047"
- board text removed: "116"
- board text removed: "232"
- board text removed: "560"
- board text removed: "DUT"

Commit message: changed pcb layout
Parts:
- added R10: 1k, Resistor_SMD:R_0805_2012Metric_Pad1.15x1.40mm_HandSolder, F.Cu at (24.6, 33.4)
- added RL4: 232, Resistor_SMD:R_0805_2012Metric_Pad1.15x1.40mm_HandSolder, F.Cu at (24.5, 45.0)
- added RL5: 232, Resistor_SMD:R_0805_2012Metric_Pad1.15x1.40mm_HandSolder, F.Cu at (24.5, 42.6)
- R7: value 60k -> 30k; footprint Resistor_SMD:R_0805_2012Metric_Pad1.15x1.40mm_HandSolder -> Resistor_SMD:R_0603_1608Metric_Pad1.05x0.95mm_HandSolder
- R8: footprint Resistor_SMD:R_0805_2012Metric_Pad1.15x1.40mm_HandSolder -> Resistor_SMD:R_0603_1608Metric_Pad1.05x0.95mm_HandSolder
- R9: value 1k -> 30k; footprint Resistor_SMD:R_0805_2012Metric_Pad1.15x1.40mm_HandSolder -> Resistor_SMD:R_0603_1608Metric_Pad1.05x0.95mm_HandSolder
- RL1: value 560 -> 232
- RL3: value 116 -> 232
- SW1: moved to B.Cu
- moved SW1 80.3 mm to (25.3, 21.6), turned to 90 degrees
- moved R9 77.2 mm to (24.6, 27.4)
- moved J2 17.1 mm to (38.7, 19.7)
- moved RL3 4.74 mm to (24.5, 47.3)
- moved RL2 4.32 mm to (24.5, 49.7)
- moved RL1 3.79 mm to (24.5, 52.0)
- moved J1 2.35 mm to (30.8, 19.6)
- moved R1 2.00 mm to (34.7, 44.8)
- moved R7 1.83 mm to (24.6, 31.2)
- moved R3 1.63 mm to (34.7, 42.5)
- moved R4 1.24 mm to (34.7, 40.1)
- moved R8 1.14 mm to (24.6, 29.3)
- moved R5 0.85 mm to (34.7, 37.7)
- moved R2 0.50 mm to (34.7, 35.4)
- moved ? 0.37 mm to (28.8, 43.2)
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Connections:
- R7 pad 2: /Vin -> Net-(R7-Pad2)
- R8 pad 1: /Vin -> Net-(R7-Pad2)
- R8 pad 2: Net-(Q5-Pad3) -> /Vin
- R9 pad 1: /SW -> /Vin
- R9 pad 2: GND -> Net-(Q5-Pad3)
- RL1 pad 2: GND -> Net-(RL1-Pad2)
- RL2 pad 1: Net-(Q2-Pad3) -> Net-(RL1-Pad2)
- RL3 pad 1: Net-(Q3-Pad3) -> Net-(Q2-Pad3)
Other:
- net class Default: clearance 0.5 -> 0.25; trace_width 0.5 -> 0.25
- rule trace_clearance: 0.5 -> 0.25
- rule trace_min: 0.5 -> 0.25

Commit message: pcb updated
Parts:
- added ?: MountingHole_3.2mm_M3_ISO7380, MountingHole:MountingHole_3.2mm_M3_ISO7380, F.Cu at (41.5, 67.3)
- added ?: MountingHole_3.2mm_M3_ISO7380, MountingHole:MountingHole_3.2mm_M3_ISO7380, F.Cu at (16.1, 67.3)
- added ?: MountingHole_3.2mm_M3_ISO7380, MountingHole:MountingHole_3.2mm_M3_ISO7380, F.Cu at (16.1, 15.2)
- added ?: MountingHole_3.2mm_M3_ISO7380, MountingHole:MountingHole_3.2mm_M3_ISO7380, F.Cu at (41.5, 15.2)
- Q5: value SI2302 -> SOT-23
- R10: value 1k -> R_0805_2012Metric_Pad1.15x1.40mm_HandSolder
- R7, R8, R9: value 30k -> R_0603_1608Metric_Pad1.05x0.95mm_HandSolder
- moved R10 0.66 mm to (23.9, 33.3)
- moved R9 0.65 mm to (23.9, 27.4)
- moved R8 0.65 mm to (23.9, 29.3)
- moved R7 0.64 mm to (23.9, 31.2)
- moved SW1 0.59 mm to (25.3, 21.0)
- moved RL1 0.21 mm to (24.3, 52.0)
- moved RL2 0.21 mm to (24.3, 49.7)
- moved RL3 0.21 mm to (24.3, 47.3)
- moved RL4 0.21 mm to (24.3, 45.0)
- moved RL5 0.21 mm to (24.3, 42.6)
Connections:
- R8 pad 1: Net-(R7-Pad2) -> /Vin
- R8 pad 2: /Vin -> Net-(R7-Pad2)
Routing:
- net /Vcc: track 0.00 -> 56.1 mm
- net /Vbat: track 0.00 -> 53.8 mm, vias 0 -> 4
- net /dut: track 0.00 -> 30.0 mm, vias 0 -> 1
- net /SW: track 0.00 -> 27.7 mm
- net /Ctrl1: track 0.00 -> 22.2 mm
- net /En_VD: track 0.00 -> 21.1 mm, vias 0 -> 1
- net /Ctrl2: track 0.00 -> 20.0 mm, vias 0 -> 1
- net /Ctrl3: track 0.00 -> 18.7 mm, vias 0 -> 1
- net /Ctrl4: track 0.00 -> 18.6 mm, vias 0 -> 1
- net Net-(D1-Pad2): track 0.00 -> 17.5 mm, vias 0 -> 1
- net /Vin: track 0.00 -> 11.9 mm, vias 0 -> 1
- net /LED4: track 0.00 -> 11.1 mm
- net Net-(Q5-Pad3): track 0.00 -> 6.87 mm
- net Net-(Q3-Pad3): track 0.00 -> 5.66 mm
- net Net-(RL1-Pad2): track 0.00 -> 3.15 mm
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- added copper zone on B.Cu, net GND
- added copper zone on F.Cu, net GND
Other:
- board outline added: 31.1 x 57.6 mm

Commit message: pcb updated
Parts:
- removed the ? at (16.1, 67.3)
- added H3: MountingHole, MountingHole:MountingHole_3.2mm_M3_ISO7380, F.Cu at (16.1, 67.3)
- ? (x3): value MountingHole_3.2mm_M3_ISO7380 -> MountingHole
- Q5: value SOT-23 -> SI2302
- R10: value R_0805_2012Metric_Pad1.15x1.40mm_HandSolder -> 1k
- R7, R8, R9: value R_0603_1608Metric_Pad1.05x0.95mm_HandSolder -> 30k
- moved SW1 0.10 mm to (25.3, 21.1)
- turned R8 to 180 degrees
Connections:
- R8 pad 1: /Vin -> Net-(R7-Pad2)
- R8 pad 2: Net-(R7-Pad2) -> /Vin
Routing:
- net /Vcc: track 56.1 -> 54.6 mm
