File: PCB_KiCAD/CapacityOfBattery.kicad_pcb (KiCad board)
At the start: 2 copper layers, 31.1 x 57.6 mm, 35 parts, among them J1 BATTERY, J2 DUT, Q1 IRLML6401TRPBF, Q2 IRLML6401TRPBF, Q3 IRLML6401TRPBF, Q4 IRLML6401TRPBF, Q5 SI2302, SW1 SW_Push

Commit message: modified pcb
Parts:
- removed ?: NodeMCU1.0(ESP-12E), lib_KiCAD:NodeMCU-LoLinV3_without_border
- removed ? (x4): MountingHole, MountingHole:MountingHole_3.2mm_M3_ISO7380
- removed ?: , lib_KiCAD:LOGO
- removed ?: KiCad-Logo2_8mm_SilkScreen, Symbol:KiCad-Logo2_8mm_SilkScreen
- removed ?: OSHW-Logo2_9.8x8mm_SilkScreen, Symbol:OSHW-Logo2_9.8x8mm_SilkScreen
- removed D1, D2, D3, D4: LED, lib_fp:LED_0805_2012Metric_Pad1.15x1.40mm_HandSolder
- removed R10: 1k, lib_fp:R_0805_2012Metric_Pad1.15x1.40mm_HandSolder
- added H1: MountingHole, lib_fp:MountingHole_3.2mm_M3_ISO7380, F.Cu at (16.1, 15.2)
- added H2: MountingHole, lib_fp:MountingHole_3.2mm_M3_ISO7380, F.Cu at (41.5, 15.2)
- added H3: MountingHole, lib_fp:MountingHole_3.2mm_M3_ISO7380, F.Cu at (16.1, 67.3)
- added H4: MountingHole, lib_fp:MountingHole_3.2mm_M3_ISO7380, F.Cu at (41.5, 67.3)
- added J3: Conn_01x04, testlibfp:128x32OLED_Display, B.Cu at (20.9, 62.0)
- added U1: NodeMCU1.0(ESP-12E), lib_fp:NodeMCU-LoLinV3_without_border, F.Cu at (28.8, 43.2)
- R2: value 560 -> 1k
- moved SW1 15.4 mm to (38.1, 29.8)
- moved R6 0.08 mm to (34.7, 33.1)
Connections:
- R2 pad 2: Net-(D1-Pad2) -> /SW
- SW1 pad 1: /Vcc -> /SW
- SW1 pad 2: /SW -> GND
Routing:
- net /Vcc: track 54.6 -> 33.8 mm
- net Net-(D1-Pad2): track 19.1 -> 0.00 mm, vias 1 -> 0
- net /Ctrl3: track 18.7 -> 4.48 mm, vias 1 -> 0
- net /Ctrl2: track 20.0 -> 7.27 mm
- net /Ctrl1: track 22.2 -> 9.63 mm
- net /Vbat: track 54.9 -> 64.1 mm
- net /LED4: track 8.62 -> 0.00 mm
- net /SW: track 27.6 -> 21.6 mm, vias 0 -> 1
- net /LED3: track 3.28 -> 0.00 mm
- net /LED2: track 3.11 -> 0.00 mm
- net /LED1: track 2.95 -> 0.00 mm
- net Net-(U1-Pad19): track 0.00 -> 1.08 mm

Commit message: modified pcb
Parts:
- moved J3 0.40 mm to (20.5, 62.0)
Routing:
- net /Vcc: track 33.8 -> 16.5 mm
Changed lines of the file:
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@@
     (thickness 1.6)
     (drawings 10)
-    (tracks 109)
+    (tracks 107)
     (zones 0)
     (modules 28)
@@
   )
   (module testlibfp:128x32OLED_Display (layer B.Cu)
-    (at 20.9 62 270)
+    (at 20.5 62 270)
     (descr "Through hole straight pin header, 1x04, 2.54mm pitch, single row")
     (tags "Through hole pin header THT 1x04 2.54mm single row")
@@
       (effects (font (size 1 1) (thickness 0.15)) (justify mirror))
     )
-    (fp_text user "128x32 OLED Display" (at -17.2 4.1 270) (layer B.SilkS)
+    (fp_text user "128x32 OLED Display" (at -17.9 -3.4 270) (layer B.SilkS)
       (effects (font (size 1 1) (thickness 0.15)) (justify mirror))
     )
@@
   (segment (start 31.79 38.93) (end 31.78 38.93) (width 0.25) (layer F.Cu) (net 4))
   (segment (start 31.78 38.93) (end 30.63 37.78) (width 0.25) (layer F.Cu) (net 4))
-  (segment (start 32.1 38.93) (end 31.78 38.93) (width 0.25) (layer F.Cu) (net 4) (status 1000000))
-  (segment (start 32.1 38.93) (end 38.89 45.72) (width 0.25) (layer B.Cu) (net 4) (status 1000000))
-  (segment (start 38.89 45.72) (end 42.81 45.72) (width 0.25) (layer B.Cu) (net 4) (status 1000000))
-  (via (at 32.1 38.93) (size 0.8) (drill 0.4) (layers F.Cu B.Cu) (net 4) (status 1000000))
+  (segment (start 32.1 38.93) (end 31.78 38.93) (width 0.25) (layer F.Cu) (net 4))
+  (segment (start 32.1 38.93) (end 38.89 45.72) (width 0.25) (layer B.Cu) (net 4))
+  (segment (start 38.89 45.72) (end 42.81 45.72) (width 0.25) (layer B.Cu) (net 4))
+  (via (at 32.1 38.93) (size 0.8) (drill 0.4) (layers F.Cu B.Cu) (net 4))
   (via (at 32 34.3) (size 0.8) (drill 0.4) (layers F.Cu B.Cu) (net 12))
   (segment (start 35.735 37.74) (end 35.735 40.1) (width 0.25) (layer F.Cu) (net 6))
@@
   (segment (start 42.59 35.4) (end 42.77 35.58) (width 0.25) (layer F.Cu) (net 6))
   (segment (start 35.725 35.4) (end 42.59 35.4) (width 0.25) (layer F.Cu) (net 6))
-  (segment (start 23.44 56.89) (end 23.44 62) (width 0.25) (layer F.Cu) (net 6))
-  (segment (start 14.83 48.28) (end 23.44 56.89) (width 0.25) (layer F.Cu) (net 6))
   (via (at 26.9 40.17) (size 0.8) (drill 0.4) (layers F.Cu B.Cu) (net 7))
   (via (at 26.9 45.27) (size 0.8) (drill 0.4) (layers F.Cu B.Cu) (net 7))

Commit message: modified pcb
Parts:
- J3: footprint testlibfp:128x32OLED_Display -> lib_fp:128x32_OLED_Display

Commit message: modified pcb
Parts:
- added ?: KiCad-Logo2_5mm_SilkScreen, Symbol:KiCad-Logo2_5mm_SilkScreen, B.Cu at (24.1, 20.6)
- added ?: OSHW-Logo2_9.8x8mm_SilkScreen, Symbol:OSHW-Logo2_9.8x8mm_SilkScreen, F.Cu at (24.3, 18.5)
- added G***: LOGO, lib_fp:test2, B.Cu at (36.5, 46.5)
- moved J3 0.24 mm to (20.4, 61.8)
Routing:
- net /Ctrl1: track 9.63 -> 51.1 mm, vias 0 -> 2
- net /SDA: track 0.00 -> 35.5 mm
- net /SCL: track 0.00 -> 34.8 mm
- net /Ctrl2: track 7.27 -> 41.8 mm, vias 1 -> 2
- net /Ctrl3: track 4.48 -> 32.2 mm, vias 0 -> 2
- net /Vcc: track 16.5 -> 43.1 mm, vias 0 -> 1
- net Net-(Q5-Pad3): track 6.87 -> 6.32 mm
- net /Vin: track 11.9 -> 12.0 mm, vias 1 -> 0

Commit message: updated images
Parts:
- G***: value LOGO -> (none); footprint lib_fp:test2 -> lib_fp:LOGO_2
