File: PCB_KiCAD/CapacityOfBattery.kicad_pcb (KiCad board)
At the start: 2 copper layers, 31.1 x 57.6 mm, 31 parts, among them J1 BATTERY, J2 DUT, J3 Conn_01x04, Q1 IRLML6401TRPBF, Q2 IRLML6401TRPBF, Q3 IRLML6401TRPBF, Q4 IRLML6401TRPBF, Q5 SI2302, SW1 SW_Push, U1 NodeMCU1.0(ESP-12E)

Commit message: updated code
Parts:
- moved G*** 0.14 mm to (36.6, 46.4)
Changed lines of the file:
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@@
       (padsonsilk false)
       (subtractmaskfromsilk false)
-      (outputformat 1)
+      (outputformat 4)
       (mirror false)
       (drillshape 0)
       (scaleselection 1)
-      (outputdirectory "gerber/"))
+      (outputdirectory "PDF/"))
   )
   (net 0 "")
@@
   )
   (module lib_fp:LOGO_2 (layer B.Cu)
-    (at 36.5 46.5 270)
+    (at 36.6 46.4 270)
     (fp_text reference G*** (at 0 0 270) (layer B.SilkS) hide
       (effects (font (size 1.524 1.524) (thickness 0.3)) (justify mirror))
@@
     (descr https://www.omron.com/ecb/products/pdf/en-b3f.pdf)
     (tags "tact sw push 6mm")
-    (fp_text reference SW1 (at 9 1.8 180) (layer B.SilkS)
+    (fp_text reference SW1 (at 3.3 2.5 270) (layer B.SilkS)
       (effects (font (size 1 1) (thickness 0.15)) (justify mirror))
     )
@@
   (segment (start 31.92 51.5) (end 30.4 53.02) (width 0.25) (layer F.Cu) (net 1))
   (via (at 31.92 51.5) (size 0.8) (drill 0.4) (layers F.Cu B.Cu) (net 1))
-  (segment (start 31.05 47.94) (end 31.9 47.09) (width 0.25) (layer F.Cu) (net 2))
-  (segment (start 30.35 47.94) (end 31.05 47.94) (width 0.25) (layer F.Cu) (net 2))
-  (segment (start 31.9 44.245) (end 33.685 42.46) (width 0.25) (layer F.Cu) (net 2))
-  (segment (start 31.9 47.09) (end 31.9 44.245) (width 0.25) (layer F.Cu) (net 2))
-  (segment (start 31.9 47.09) (end 31.9 47.09) (width 0.25) (layer F.Cu) (net 2))
-  (segment (start 33.16 40.1) (end 33.685 40.1) (width 0.25) (layer F.Cu) (net 3))
-  (segment (start 30.4 42.86) (end 32.16 41.1) (width 0.25) (layer F.Cu) (net 3))
-  (segment (start 30.35 42.86) (end 30.4 42.86) (width 0.25) (layer F.Cu) (net 3))
-  (segment (start 33.645 37.78) (end 33.685 37.74) (width 0.25) (layer F.Cu) (net 4))
-  (segment (start 30.63 37.78) (end 33.645 37.78) (width 0.25) (layer F.Cu) (net 4))
-  (segment (start 31.79 38.93) (end 31.78 38.93) (width 0.25) (layer F.Cu) (net 4))
-  (segment (start 31.78 38.93) (end 30.63 37.78) (width 0.25) (layer F.Cu) (net 4))
-  (segment (start 32.1 38.93) (end 31.78 38.93) (width 0.25) (layer F.Cu) (net 4))
-  (segment (start 32.1 38.93) (end 38.89 45.72) (width 0.25) (layer B.Cu) (net 4))
-  (segment (start 38.89 45.72) (end 42.81 45.72) (width 0.25) (layer B.Cu) (net 4))
-  (via (at 32.1 38.93) (size 0.8) (drill 0.4) (layers F.Cu B.Cu) (net 4))
   (via (at 29 26.5) (size 0.8) (drill 0.4) (layers F.Cu B.Cu) (net 1))
   (segment (start 31.92 50.934315) (end 31.92 51.5) (width 0.25) (layer B.Cu) (net 1))
@@
   (segment (start 40.15 25.5) (end 42.77 22.88) (width 0.25) (layer F.Cu) (net 1))
   (segment (start 30 25.5) (end 40.15 25.5) (width 0.25) (layer F.Cu) (net 1))
+  (segment (start 31.05 47.94) (end 31.9 47.09) (width 0.25) (layer F.Cu) (net 2))
+  (segment (start 30.35 47.94) (end 31.05 47.94) (width 0.25) (layer F.Cu) (net 2))
+  (segment (start 31.9 44.245) (end 33.685 42.46) (width 0.25) (layer F.Cu) (net 2))
+  (segment (start 31.9 47.09) (end 31.9 44.245) (width 0.25) (layer F.Cu) (net 2))
+  (segment (start 31.9 47.09) (end 31.9 47.09) (width 0.25) (layer F.Cu) (net 2))
   (via (at 30.1 27.5) (size 0.8) (drill 0.4) (layers F.Cu B.Cu) (net 2))
   (segment (start 31.9 47.09) (end 31.9 47.09) (width 0.25) (layer F.Cu) (net 2))
@@
   (segment (start 42.77 25.42) (end 41.59 26.6) (width 0.25) (layer F.Cu) (net 2))
   (segment (start 41.59 26.6) (end 41.39 26.8) (width 0.25) (layer F.Cu) (net 2))
+  (segment (start 33.16 40.1) (end 33.685 40.1) (width 0.25) (layer F.Cu) (net 3))
+  (segment (start 30.4 42.86) (end 32.16 41.1) (width 0.25) (layer F.Cu) (net 3))
+  (segment (start 30.35 42.86) (end 30.4 42.86) (width 0.25) (layer F.Cu) (net 3))
   (segment (start 42.77 27.96) (end 37.2 33.53) (width 0.25) (layer F.Cu) (net 3))
   (segment (start 37.2 33.53) (end 37.2 46.2) (width 0.25) (layer F.Cu) (net 3))
@@
   (segment (start 37.2 46.14) (end 37.2 46.2) (width 0.25) (layer B.Cu) (net 3))
   (segment (start 32.16 41.1) (end 37.2 46.14) (width 0.25) (layer B.Cu) (net 3))
+  (segment (start 33.645 37.78) (end 33.685 37.74) (width 0.25) (layer F.Cu) (net 4))
+  (segment (start 30.63 37.78) (end 33.645 37.78) (width 0.25) (layer F.Cu) (net 4))
+  (segment (start 31.79 38.93) (end 31.78 38.93) (width 0.25) (layer F.Cu) (net 4))
+  (segment (start 31.78 38.93) (end 30.63 37.78) (width 0.25) (layer F.Cu) (net 4))
+  (segment (start 32.1 38.93) (end 31.78 38.93) (width 0.25) (layer F.Cu) (net 4))
+  (segment (start 32.1 38.93) (end 38.89 45.72) (width 0.25) (layer B.Cu) (net 4))
+  (segment (start 38.89 45.72) (end 42.81 45.72) (width 0.25) (layer B.Cu) (net 4))
+  (via (at 32.1 38.93) (size 0.8) (drill 0.4) (layers F.Cu B.Cu) (net 4))
   (segment (start 35.735 37.74) (end 35.735 40.1) (width 0.25) (layer F.Cu) (net 6))
   (segment (start 35.735 40.1) (end 35.735 42.46) (width 0.25) (layer F.Cu) (net 6))

Commit message: update README
Other:
- board text added: "mAhTime"
Changed lines of the file:
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@@
   (general
     (thickness 1.6)
-    (drawings 10)
+    (drawings 11)
     (tracks 154)
     (zones 0)
@@
       (padsonsilk false)
       (subtractmaskfromsilk false)
-      (outputformat 4)
+      (outputformat 1)
       (mirror false)
       (drillshape 0)
       (scaleselection 1)
-      (outputdirectory "PDF/"))
+      (outputdirectory "gerber/"))
   )
   (net 0 "")
@@
       (xy -3.43224 2.584467) (xy -3.324904 2.572722) (xy -3.231114 2.584505)) (layer F.SilkS) (width 0.01))
   )
+  (gr_text mAhTime (at 29.2 15) (layer B.SilkS)
+    (effects (font (size 1.5 1.5) (thickness 0.3)) (justify mirror))
+  )
   (gr_text appiko.org (at 28.702 67.183) (layer F.SilkS)
     (effects (font (size 1.5 1.5) (thickness 0.3)))
   )
   (gr_text "v 1.0" (at 28.9 67.4) (layer B.SilkS)
-    (effects (font (size 1.5 1.5) (thickness 0.3)) (justify mirror))
+    (effects (font (size 1 1) (thickness 0.15)) (justify mirror))
   )
   (gr_arc (start 16.1 67.2) (end 13.3 67.2) (angle -90) (layer Edge.Cuts) (width 0.1))
